Commit message: test(armkit): extend meshed.urdf and update its mesh-count assertion
meshed.urdf now references 3 mesh files, not 2 (see previous commit's
mesh-inspection tests for why): update the one place that hardcoded the
old count.

File: skills/viam-arm-module/scripts/tests/fixtures/meshed.urdf (robot description, URDF)
Before this commit: robot meshed, 2 links, 1 joints
Links:
- link link1: geometry collision mesh filename=meshes/link1.stl; visual mesh filename=meshes/link1.dae
